Commit message: done control teleop

File: mybot_description/urdf/macros.xacro (robot description, xacro)
@@ -1,67 +1,66 @@
 <?xml version="1.0"?>
 <robot>
-   <macro name="cylinder_inertia" params="m r h">
-   <inertia  ixx="${m*(3*r*r+h*h)/12}" ixy = "0" ixz = "0"
-      iyy="${m*(3*r*r+h*h)/12}" iyz = "0"
-      izz="${m*r*r/2}"
-   />
-   </macro>
-   <macro name="box_inertia" params="m x y z">
-   <inertia  ixx="${m*(y*y+z*z)/12}" ixy = "0" ixz = "0"
-      iyy="${m*(x*x+z*z)/12}" iyz = "0"
-      izz="${m*(x*x+z*z)/12}"
-   />
-   </macro>
-   <macro name="sphere_inertia" params="m r">
-   <inertia  ixx="${2*m*r*r/5}" ixy = "0" ixz = "0"
-      iyy="${2*m*r*r/5}" iyz = "0"
-      izz="${2*m*r*r/5}"
-   />
-   </macro>
-   <macro name="wheel" params="lr tY">
-      <link name="${lr}_wheel">
-         <collision>
-            <origin xyz="0 0 0" rpy="0 ${PI/2} ${PI/2}" />
-            <geometry>
-               <cylinder length="${wheelWidth}" radius="${wheelRadius}"/>
-            </geometry>
-         </collision>
-         <visual>
-            <origin xyz="0 0 0" rpy="0 ${PI/2} ${PI/2}" />
-            <geometry>
-               <cylinder length="${wheelWidth}" radius="${wheelRadius}"/>
-            </geometry>
-            <material name="black"/>
-         </visual>
-         <inertial>
-            <origin xyz="0 0 0" rpy="0 ${PI/2} ${PI/2}" />
-            <mass value="${wheelMass}"/>
-            <cylinder_inertia m="${wheelMass}" r="${wheelRadius}" h="${wheelWidth}"/>
-         </inertial>
-      </link>
-      <gazebo reference="${lr}_wheel">
-         <mu1 value="1.0"/>
-         <mu2 value="1.0"/>
-         <kp  value="10000000.0" />
-         <kd  value="1.0" />
-         <fdir1 value="1 0 0"/>
-         <material>Gazebo/Black</material>
-      </gazebo>
-      <joint name="${lr}_wheel_hinge" type="continuous">
-      <parent link="chassis"/>
-      <child link="${lr}_wheel"/>
-      <origin xyz="${-wheelPos+chassisLength/2} ${tY*wheelWidth/2+tY*chassisWidth/2} ${wheelRadius}" rpy="0 0 0" />
-      <axis xyz="0 1 0" rpy="0 0 0" />
-      <limit effort="100" velocity="100"/>
-      <joint_properties damping="0.0" friction="0.0"/>
-      </joint>
+     <macro name="cylinder_inertia" params="m r h">
+        <inertia  ixx="${m*(3*r*r+h*h)/12}" ixy = "0" ixz = "0"
+                  iyy="${m*(3*r*r+h*h)/12}" iyz = "0"
+                  izz="${m*r*r/2}" />
+      </macro>
+      <macro name="box_inertia" params="m x y z">
+        <inertia  ixx="${m*(y*y+z*z)/12}" ixy = "0" ixz = "0"
+                  iyy="${m*(x*x+z*z)/12}" iyz = "0"
+                  izz="${m*(x*x+z*z)/12}" />
+      </macro>
+      <macro name="sphere_inertia" params="m r">
+        <inertia  ixx="${2*m*r*r/5}" ixy = "0" ixz = "0"
+                  iyy="${2*m*r*r/5}" iyz = "0"
+                  izz="${2*m*r*r/5}" />
+      </macro>
+     <macro name="wheel" params="lr tY">
+       <link name="${lr}_wheel">
+        <collision>
+          <origin xyz="0 0 0" rpy="0 ${PI/2} ${PI/2}" />
+          <geometry>
+           <cylinder length="${wheelWidth}" radius="${wheelRadius}"/>
+          </geometry>
+        </collision>
+        <visual>
+          <origin xyz="0 0 0" rpy="0 ${PI/2} ${PI/2}" />
+          <geometry>
+           <cylinder length="${wheelWidth}" radius="${wheelRadius}"/>
+          </geometry>
+          <material name="black"/>
+        </visual>
+        <inertial>
+          <origin xyz="0 0 0" rpy="0 ${PI/2} ${PI/2}" />
+          <mass value="${wheelMass}"/>
+          <cylinder_inertia m="${wheelMass}" r="${wheelRadius}" h="${wheelWidth}"/>
+        </inertial>
+       </link>
+        <gazebo reference="${lr}_wheel">
+          <mu1 value="1.0"/>
+          <mu2 value="1.0"/>
+          <kp  value="10000000.0" />
+          <kd  value="1.0" />
+          <fdir1 value="1 0 0"/>
+          <material>Gazebo/Black</material>
+        </gazebo>
+       <joint name="${lr}_wheel_hinge" type="continuous">
+          <parent link="chassis"/>
+          <child link="${lr}_wheel"/>
+          <origin xyz="${+wheelPos-chassisLength/4} ${tY*wheelWidth/2+tY*chassisWidth/2} ${wheelRadius}" rpy="0 0 0" />
+          <axis xyz="0 1 0" rpy="0 0 0" />
+          <limit effort="600" velocity="600"/>
+          <!-- <joint_properties damping="0.0" friction="0.0"/> -->
+        </joint>
       <transmission name="${lr}_trans">
-      <type>transmission_interface/SimpleTransmission</type>
-      <joint name="${lr}_wheel_hinge"/>
-      <actuator name="${lr}Motor">
-         <hardwareInterface>EffortJointInterface</hardwareInterface>
-         <mechanicalReduction>10</mechanicalReduction>
-      </actuator>
+        <type>transmission_interface/SimpleTransmission</type>
+        <joint name="${lr}_wheel_hinge">
+            <hardwareInterface>hardware_interface/EffortJointInterface</hardwareInterface>
+        </joint>
+        <actuator name="${lr}Motor">
+             <hardwareInterface>hardware_interface/EffortJointInterface</hardwareInterface>
+          <mechanicalReduction>10</mechanicalReduction>
+        </actuator>
       </transmission>
-   </macro>
+     </macro>
 </robot>

File: mybot_description/urdf/mybot.xacro (robot description, xacro)
@@ -50,5 +50,5 @@
       <origin xyz="${casterRadius-chassisLength/2} 0 ${casterRadius-chassisHeight+wheelRadius}" rpy="0 0 0"/>
       <geometry>
-	<sphere radius="${casterRadius}"/>
+	      <sphere radius="${casterRadius}"/>
       </geometry>
     </collision>
@@ -56,5 +56,5 @@
       <origin xyz="${casterRadius-chassisLength/2} 0 ${casterRadius-chassisHeight+wheelRadius}" rpy="0 0 0"/>
       <geometry>
-	<sphere radius="${casterRadius}"/>
+	      <sphere radius="${casterRadius}"/>
       </geometry>
     </visual>

Commit message: error pub

File: mybot_description/urdf/macros.xacro (robot description, xacro)
@@ -50,5 +50,5 @@
           <origin xyz="${+wheelPos-chassisLength/4} ${tY*wheelWidth/2+tY*chassisWidth/2} ${wheelRadius}" rpy="0 0 0" />
           <axis xyz="0 1 0" rpy="0 0 0" />
-          <limit effort="600" velocity="600"/>
+          <limit effort="100" velocity="100"/>
           <!-- <joint_properties damping="0.0" friction="0.0"/> -->
         </joint>

File: mybot_description/urdf/mybot.xacro (robot description, xacro)
@@ -26,5 +26,5 @@
       <origin xyz="0 0 ${wheelRadius}" rpy="0 0 0"/>
       <geometry>
-	<box size="${chassisLength} ${chassisWidth} ${chassisHeight}"/>
+        <box size="${chassisLength} ${chassisWidth} ${chassisHeight}"/>
       </geometry>
     </collision>
@@ -32,5 +32,5 @@
       <origin xyz="0 0 ${wheelRadius}" rpy="0 0 0"/>
       <geometry>
-	<box size="${chassisLength} ${chassisWidth} ${chassisHeight}"/>
+        <box size="${chassisLength} ${chassisWidth} ${chassisHeight}"/>
       </geometry>
       <material name="orange"/>
@@ -67,3 +67,23 @@
   <wheel lr="left" tY="-1"/>
   <wheel lr="right" tY="1"/>
+  <!-- <link name="camera">
+    <collision>
+      <origin xyz="0 0 0" rpy="0 0 0"/>
+      <geometry>
+        <box size="${cameraSize} ${cameraSize} ${cameraSize}"/>
+      </geometry>
+    </collision>
+    <visual>
+      <origin xyz="0 0 0" rpy="0 0 0"/>
+      <geometry>
+        <box size="${cameraSize} ${cameraSize} ${cameraSize}"/>
+      </geometry>
+      <material name="blue"/>
+    </visual>
+    <inertial>
+      <mass value="${cameraMass}" />
+      <origin xyz="0 0 0" rpy="0 0 0"/>
+      <box_inertia m="${cameraMass}" x="${cameraSize}" y="${cameraSize}" z="${cameraSize}" />
+    </inertial>
+  </link> -->
 </robot>
